File: Hardware/KiCad/RPROM.kicad_sch (KiCad schematic)
At the start: 41 parts, among them IC1 W25Q32JVZP, J1 USB_B_Micro, J2 Conn_01x20, J3 Conn_01x20, J4 Conn_01x01, SW1 SW_Push, SW2 SW_Push, U1 RP2350_80QFN, U2 TLV1117-33, Y1 ABM8-272-T3

Commit message: Update KiCad design to use correct flash component
Parts:
- IC1: value W25Q32JVZP -> W25Q32RVXHJQ; symbol Memory_Flash:W25Q32JVZP -> RPROM:W25Q32RVXHJQ
Changed lines of the file:
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@@
 	)
 	(symbol
-		(lib_id "Memory_Flash:W25Q32JVZP")
+		(lib_id "RPROM:W25Q32RVXHJQ")
 		(at 67.31 189.23 0)
 		(unit 1)
@@
 			)
 		)
-		(property "Value" "W25Q32JVZP"
+		(property "Value" "W25Q32RVXHJQ"
 			(at 76.2 190.4999 0)
 			(effects
@@
 			)
 		)
-		(property "Datasheet" "http://www.winbond.com/resource-files/w25q32jv%20revg%2003272018%20plus.pdf"
+		(property "Datasheet" "https://www.winbond.com/hq/product/code-storage-flash-memory/serial-nor-flash/?__locale=en&partNo=W25Q32RV"
 			(at 67.31 191.77 0)
 			(effects
@@
 			)
 		)
-		(property "Description" "32Mb Serial Flash Memory, Standard/Dual/Quad SPI, DFN-8"
+		(property "Description" "NOR Flash spiFlash, 3V, 32M-bit, 4Kb Uniform Sector"
 			(at 67.31 189.23 0)
 			(effects
